File: PD65W_Charger.kicad_sch (KiCad schematic)
At the start: 27 parts, among them J1 Barrel_Jack_MountingPin, J2 Output_V-from-PD65, J3 FAN, Q1 2N2222, U2 OLED_0.91-I2C, U3 MOUDLE-SEEEDUINO-XIAO, U4 AP63205WU, U5 INA226

Commit message: Created README.md with BOM
Parts:
- added C6: 10µF 50V, Capacitor_SMD:C_0805_2012Metric_Pad1.18x1.45mm_HandSolder, symbol Device:C
- C2: value 10µF 50V -> 10µF 35V
- C4: footprint Capacitor_SMD:C_0805_2012Metric -> Capacitor_SMD:C_0805_2012Metric_Pad1.18x1.45mm_HandSolder
- C5: value C -> 100nF
- D1: value D_Schottky -> 1N4148
- J1: footprint Connector_BarrelJack:BarrelJack_GCT_DCJ200-10-A_Horizontal -> Connector_BarrelJack:BarrelJack_Horizontal
- L1: footprint Inductor_SMD:L_Bourns-SRN4018 -> Inductor_SMD:L_6.3x6.3_H3
- U1: value (none) -> PD65W_module
Connections:
- net +24V: now also C6.2
- net GND: now also C6.1
Other:
- moved on the sheet: C2
