File: PD65W_Charger.kicad_pcb (KiCad board)
At the start: 2 copper layers, 27 parts, among them J1 Barrel_Jack_MountingPin, J2 Output_V-from-PD65, J3 FAN, Q1 2N2222, U2 OLED_0.91-I2C, U3 MOUDLE-SEEEDUINO-XIAO, U4 AP63205WU, U5 INA226

Commit message: Created README.md with BOM
Parts:
- moved U2 17.5 mm to (110.6, 71.4)
- moved U1 2.30 mm to (132.6, 84.5)
Other:
- board outline added: 18.5 x 12.8 mm
Changed lines of the file:
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@@
 	(footprint "Library_footprint:PD65W_module"
 		(layer "F.Cu")
-		(at 131.76 82.29)
+		(at 132.55 84.45)
 		(property "Reference" "U1"
 			(at 0 -0.5 0)
@@
 		(sheetname "/")
 		(sheetfile "PD65W_Charger.kicad_sch")
+		(units
+			(unit
+				(name "A")
+				(pins "1" "2")
+			)
+		)
 		(attr smd)
 		(duplicate_pad_numbers_are_jumpers no)
@@
 		)
 		(fp_rect
+			(start -9.27 -6.42)
+			(end 9.27 6.42)
+			(radius 2)
+			(stroke
+				(width 0.05)
+				(type solid)
+			)
+			(fill no)
+			(layer "Edge.Cuts")
+		)
+		(fp_rect
 			(start -12.23 -9.24)
 			(end 12.28 9.25)
@@
 			(fill no)
 			(layer "F.Fab")
+		)
+		(fp_text user "+"
+			(at 11.96 -6.6 0)
+			(unlocked yes)
+			(layer "F.SilkS")
+			(effects
+				(font
+					(size 2 2)
+				)
+				(justify left bottom)
+			)
+		)
+		(fp_text user "-"
+			(at 11.96 8.89 0)
+			(unlocked yes)
+			(layer "F.SilkS")
+			(effects
+				(font
+					(size 2 2)
+				)
+				(justify left bottom)
+			)
 		)
 		(fp_text user "${REFERENCE}"
@@
 	(footprint "Display:ER_OLEDM0.91_1x-I2C"
 		(layer "F.Cu")
-		(at 122.425 58.495 90)
+		(at 110.6 71.41 90)
 		(descr "SSD1306 OLED module, 0.91 inch, 128x32, I2C (https://www.buydisplay.com/download/manual/ER-OLEDM0.91-1_Datasheet.pdf)")
 		(tags "EastRising")

Commit message: Added order_35321745.csv that can be imported to TME.eu that will automatically import all product to cart
Parts:
- added C6: 10µF 50V, Capacitor_SMD:C_0805_2012Metric_Pad1.18x1.45mm_HandSolder, F.Cu at (149.8, 108.6)
- C2: value 10µF 50V -> 10µF 35V
- C4: footprint Capacitor_SMD:C_0805_2012Metric -> Capacitor_SMD:C_0805_2012Metric_Pad1.18x1.45mm_HandSolder
- C5: value C -> 100nF
- D1: value D_Schottky -> 1N4148
- J1: footprint Connector_BarrelJack:BarrelJack_GCT_DCJ200-10-A_Horizontal -> Connector_BarrelJack:BarrelJack_Horizontal
- L1: footprint Inductor_SMD:L_Bourns-SRN4018 -> Inductor_SMD:L_6.3x6.3_H3
- U1: value ~ -> PD65W_module
- moved J1 9.67 mm to (159.0, 98.8)
Other:
- board size 18.5 x 12.8 mm -> 84.6 x 64.4 mm

Commit message: upload
Parts:
- R1: moved to B.Cu
- moved U2 69.6 mm to (168.0, 110.8), turned to 180 degrees
- moved TH1 47.0 mm to (174.5, 76.0)
- moved U3 46.7 mm to (180.5, 104.4), turned to -90 degrees
- moved R2 41.5 mm to (174.0, 80.0)
- moved R3 39.0 mm to (166.7, 106.8), turned to -90 degrees
- moved TH2 37.3 mm to (165.5, 86.5), turned to 180 degrees
- moved R4 37.2 mm to (168.6, 106.8), turned to -90 degrees
- moved Q1 36.8 mm to (152.8, 108.3), turned to 90 degrees
- moved R8 31.6 mm to (157.2, 113.6), turned to 180 degrees
- moved J2 29.2 mm to (150.4, 98.4)
- moved C6 28.3 mm to (169.5, 88.2), turned to 90 degrees
- moved R1 26.1 mm to (164.5, 89.5)
- moved R9 24.9 mm to (157.0, 109.8), turned to -90 degrees
- moved J1 22.9 mm to (177.0, 84.7), turned to 180 degrees
- moved R6 22.0 mm to (154.6, 98.4)
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Connections:
- R1 pad 2: /A0 -> /A1
- R2 pad 2: /A1 -> /A0
- R8 pad 1: /D3 -> /D10
- U3 pad 10: unconnected-(U3-PA5_A9_D9_MISO-Pad10)_1 -> /D10
- U3 pad 4: /D3 -> unconnected-(U3-PA11_A3_D3-Pad4)_1
Routing:
- net +5V: track 0.00 -> 138.7 mm
- net +3V3: track 0.00 -> 93.0 mm, vias 0 -> 3
- net +24V: track 0.00 -> 38.1 mm
- net /A2: track 0.00 -> 36.4 mm
- net /SDA: track 0.00 -> 29.8 mm
- net /SCL: track 0.00 -> 28.7 mm, vias 0 -> 2
- net /A0: track 0.00 -> 27.9 mm
- net /A1: track 0.00 -> 27.1 mm, vias 0 -> 1
- net /D10: track 0.00 -> 21.7 mm
- net Net-(D1-A): track 0.00 -> 13.2 mm
- net Net-(Q1-B): track 0.00 -> 10.9 mm
- net Net-(U1-IN+): track 0.00 -> 9.87 mm
- net Net-(U4-SW): track 0.00 -> 8.60 mm
- net Net-(J2-Pin_1): track 0.00 -> 3.20 mm
- net Net-(U4-BST): track 0.00 -> 2.90 mm
- added copper zone on B.Cu, net GND
- added copper zone on F.Cu, net GND
Other:
- board size 84.6 x 64.4 mm -> 50.9 x 44.4 mm
