File: PD65W_Charger.kicad_pcb (KiCad board)
At the start: 2 copper layers, 50.9 x 44.4 mm, 28 parts, among them J1 Barrel_Jack_MountingPin, J2 Output_V-from-PD65, J3 FAN, Q1 2N2222, U1 PD65W_module, U2 OLED_0.91-I2C, U3 MOUDLE-SEEEDUINO-XIAO, U4 AP63205WU, U5 INA226

Commit message: Everything exccept Documentation done
Parts:
- added H1: MountingHole, MountingHole:MountingHole_3.2mm_M3_DIN965, F.Cu at (187.2, 75.3)
- moved J3 0.91 mm to (144.0, 99.0)
Routing:
- net Net-(D1-A): track 13.2 -> 12.2 mm
Changed lines of the file:
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@@
 	(footprint "Connector_PinHeader_2.54mm:PinHeader_1x02_P2.54mm_Vertical"
 		(layer "F.Cu")
-		(at 143.225 98.5 90)
+		(at 143.97 99.02 90)
 		(descr "Through hole straight pin header, 1x02, 2.54mm pitch, single row")
 		(tags "Through hole pin header THT 1x02 2.54mm single row")
@@
 		(attr smd)
 		(duplicate_pad_numbers_are_jumpers no)
+		(fp_line
+			(start -12.1 0)
+			(end -10.25 0)
+			(stroke
+				(width 0.25)
+				(type solid)
+			)
+			(layer "F.SilkS")
+		)
 		(fp_rect
 			(start -12.1 -9.1)
@@
 		)
 	)
+	(footprint "MountingHole:MountingHole_3.2mm_M3_DIN965"
+		(layer "F.Cu")
+		(at 187.25 75.26)
+		(descr "Mounting Hole 3.2mm, M3, no annular, generated by kicad-footprint-generator mountinghole.py")
+		(tags "mountinghole M3 DIN965")
+		(property "Reference" "H1"
+			(at 0 -3.75 0)
+			(layer "F.SilkS")
+			(effects
+				(font
+					(size 1 1)
+					(thickness 0.15)
+				)
+			)
+		)
+		(property "Value" "MountingHole"
+			(at 0 3.75 0)
+			(layer "F.Fab")
+			(effects
+				(font
+					(size 1 1)
+					(thickness 0.15)
+				)
+			)
+		)
+		(property "Datasheet" ""
+			(at 0 0 0)
+			(layer "F.Fab")
+			(hide yes)
+			(effects
+				(font
+					(size 1.27 1.27)
+				)
+			)
+		)
+		(property "Description" "Mounting Hole without connection"
+			(at 0 0 0)
+			(layer "F.Fab")
+			(hide yes)
+			(effects
+				(font
+					(size 1.27 1.27)
+				)
+			)
+		)
+		(property "KiLib_Generator" "mounting_hardware/mounting_hole"
+			(at 0 0 0)
+			(layer "F.SilkS")
+			(hide yes)
+			(effects
+				(font
+					(size 1 1)
+					(thickness 0.15)
+				)
+			)
+		)
+		(property ki_fp_filters "MountingHole*")
+		(sheetname "/")
+		(sheetfile "PD65W_Charger.kicad_sch")
+		(units
+			(unit
+				(name "A")
+				(pins)
+			)
+		)
+		(attr exclude_from_bom)
+		(duplicate_pad_numbers_are_jumpers no)
+		(fp_circle
+			(center 0 0)
+			(end 2.8 0)
+			(stroke
+				(width 0.15)
+				(type solid)
+			)
+			(fill no)
+			(layer "Cmts.User")
+		)
+		(fp_circle
+			(center 0 0)
+			(end 3.05 0)
+			(stroke
+				(width 0.05)
+				(type solid)
+			)
+			(fill no)
+			(layer "F.CrtYd")
+		)
+		(fp_text user "${REFERENCE}"
+			(at 0 0 0)
+			(layer "F.Fab")
+			(effects
+				(font
+					(size 1 1)
+					(thickness 0.15)
+				)
+			)
+		)
+		(pad "" np_thru_hole circle
+			(at 0 0)
+			(size 3.2 3.2)
+			(drill 3.2)
+			(layers "*.Cu" "*.Mask")
+		)
+		(embedded_fonts no)
+	)
 	(footprint "Package_TO_SOT_THT:TO-92"
 		(layer "F.Cu")
@@
 		(sheetname "/")
 		(sheetfile "PD65W_Charger.kicad_sch")
+		(units
+			(unit
+				(name "A")
+				(pins "3" "4" "2" "1")
+			)
+		)
 		(attr through_hole)
 		(duplicate_pad_numbers_are_jumpers no)
@@
 		)
 		(embedded_fonts no)
-		(model "${KICAD10_3DMODEL_DIR}/Display.3dshapes/ER_OLEDM0.91_1x-I2C.step"
+		(model "${KIPRJMOD}/other_libraries/3d_models/OLED_0.91_128x32.stp"
 			(offset
-				(xyz 0 0 0)
+				(xyz 3.8 -17.5 6.5)
 			)
 			(scale
@@
 			)
 			(rotate
-				(xyz 0 0 0)
+				(xyz -0 -0 90)
 			)
 		)
@@
 		)
 		(embedded_fonts no)
-		(model "${AMZPATH}/3dmodels/AMz3D.3dshapes/XIAO-nRF52840 v15.step"
-			(hide yes)
-			(offset
-				(xyz -1.778 -6.096 0.381)
-			)
-			(scale
-				(xyz 1 1 1)
-			)
-			(rotate
-				(xyz -90 0 0)
-			)
-		)
-		(model "${AMZPATH}/3dmodels/AMz3D.3dshapes/Seeeduino XIAO SAMD21 v4.step"
+		(model "${KIPRJMOD}/other_libraries/3d_models/Seeed Studio XIAO RP2040 v26.step"
 			(offset
 				(xyz 0 0 0)
@@
 			)
 		)
-		(model "${AMZPATH}/3dmodels/AMz3D.3dshapes/Seeed Studio XIAO RP2040 v26.step"
-			(hide yes)
-			(offset
-				(xyz 0 0 0)
-			)
-			(scale
-				(xyz 1 1 1)
-			)
-			(rotate
-				(xyz 0 0 90)
-			)
-		)
-		(model "${AMZPATH}/3dmodels/AMz3D.3dshapes/Seeed Studio XIAO-ESP32-C3.step"
-			(hide yes)
-			(offset
-				(xyz -1.7018 -6.096 0)
-			)
-			(scale
-				(xyz 1 1 1)
-			)
-			(rotate
-				(xyz -90 0 0)
-			)
-		)
-		(model "${AMZPATH}/3dmodels/AMz3D.3dshapes/XIAO-ESP32S3 v2.step"
-			(hide yes)
-			(offset
-				(xyz -1.778 -6.1722 0)
-			)
-			(scale
-				(xyz 1 1 1)
-			)
-			(rotate
-				(xyz -90 0 0)
-			)
-		)
 	)
 	(footprint "Inductor_SMD:L_6.3x6.3_H3"
@@
 	)
 	(gr_line
-		(start 136 97)
-		(end 136 72)
-		(stroke
-			(width 0.2)
-			(type solid)
-		)
-		(layer "Dwgs.User")
-	)
-	(gr_line
 		(start 140.2 71.375)
 		(end 140.2 102)
@@
 	)
 	(segment
-		(start 178.575 72.175)
-		(end 163.225 72.175)
-		(width 0.6)
+		(start 143.225 99.765)
+		(end 143.97 99.02)
+		(width 0.45)
 		(layer "F.Cu")
 		(net "+5V")
 	)
 	(segment
-		(start 143.225 101.425)
-		(end 143.225 98.5)
-		(width 0.45)
+		(start 178.575 72.175)
+		(end 163.225 72.175)
+		(width 0.6)
 		(layer "F.Cu")
 		(net "+5V")
@@
 	)
 	(segment
-		(start 144.2 102.4)
-		(end 143.225 101.425)
+		(start 146 102.4)
+		(end 144.2 102.4)
 		(width 0.45)
 		(layer "F.Cu")
@@
 	)
 	(segment
+		(start 143.225 101.425)
+		(end 143.225 99.765)
+		(width 0.45)
+		(layer "F.Cu")
+		(net "+5V")
+	)
+	(segment
 		(start 186.2 79.8)
 		(end 178.575 72.175)
@@
 	)
 	(segment
-		(start 146 102.4)
-		(end 144.2 102.4)
+		(start 144.2 102.4)
+		(end 143.225 101.425)
 		(width 0.45)
 		(layer "F.Cu")
@@
 	)
 	(segment
+		(start 147.58 99.02)
+		(end 150.96 102.4)
+		(width 0.25)
+		(layer "F.Cu")
+		(net "Net-(D1-A)")
+	)
+	(segment
 		(start 152.77 105.73)
 		(end 153.62 104.88)
@@
 	)
 	(segment
-		(start 147.1 98.5)
-		(end 151 102.4)
+		(start 150.96 102.4)
+		(end 153.62 102.4)
 		(width 0.25)
 		(layer "F.Cu")
@@
 	)
 	(segment
-		(start 151 102.4)
-		(end 153.62 102.4)
+		(start 146.51 99.02)
+		(end 147.58 99.02)
 		(width 0.25)
 		(layer "F.Cu")
@@
 	)
 	(segment
-		(start 145.765 98.5)
-		(end 147.1 98.5)
-		(width 0.25)
-		(layer "F.Cu")
-		(net "Net-(D1-A)")
-	)
-	(segment
 		(start 169.274749 96.925251)
 		(end 168.8 97.4)
@@
 	)
 	(via
-		(at 187.24 77.8)
+		(at 182.92 73.68)
 		(size 0.6)
 		(drill 0.4)
