File: _restore_backup_2026-08-26T09-27-49-905/PD65W_Charger.kicad_sch (KiCad schematic)
At the start: 28 parts, among them J1 Barrel_Jack_MountingPin, J2 Output_V-from-PD65, J3 FAN, Q1 2N2222, U1 PD65W_module, U2 OLED_0.91-I2C, U3 MOUDLE-SEEEDUINO-XIAO, U4 AP63205WU, U5 INA226

Commit message: upload
Connections:
- net A0: now also R1.2; no longer R2.2
- net A1: now also R2.2; no longer R1.2
- net D3: now reaches U3.4 (PA11_A3_D3)
- net D3: now also R8.1
- net D10: no longer names the net of U3.10 (PA5_A9_D9_MISO)
- net D10: no longer R8.1
Other:
- moved on the sheet: R2
Changed lines of the file:
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@@
 	)
 	(junction
-		(at 128.27 137.16)
+		(at 71.12 49.53)
 		(diameter 0)
 		(color 0 0 0 0)
 	)
 	(junction
-		(at 138.43 116.84)
+		(at 128.27 137.16)
 		(diameter 0)
 		(color 0 0 0 0)
 	)
 	(junction
-		(at 128.27 134.62)
+		(at 138.43 116.84)
 		(diameter 0)
 		(color 0 0 0 0)
 	)
 	(junction
-		(at 71.12 49.53)
+		(at 128.27 134.62)
 		(diameter 0)
 		(color 0 0 0 0)
@@
 	)
 	(no_connect
-		(at 109.22 44.45)
+		(at 152.4 46.99)
 	)
 	(no_connect
@@
 	(wire
 		(pts
-			(xy 153.67 46.99) (xy 152.4 46.99)
-		)
-		(stroke
-			(width 0)
-			(type default)
-		)
-	)
-	(wire
-		(pts
 			(xy 148.59 132.08) (xy 151.13 132.08)
 		)
@@
 		)
 	)
-	(label "D10"
+	(label "D3"
 		(at 66.04 133.35 180)
 		(effects
@@
 		)
 	)
-	(label "D10"
-		(at 153.67 46.99 0)
+	(label "D3"
+		(at 109.22 44.45 180)
 		(effects
 			(font
 				(size 1.27 1.27)
 			)
-			(justify left bottom)
+			(justify right bottom)
 		)
 	)
@@
 	)
 	(symbol
+		(lib_id "Device:R")
+		(at 44.45 43.18 0)
+		(unit 1)
+		(body_style 1)
+		(exclude_from_sim no)
+		(in_bom yes)
+		(on_board yes)
+		(in_pos_files yes)
+		(dnp no)
+		(fields_autoplaced yes)
+		(property "Reference" "R1"
+			(at 46.99 41.9099 0)
+			(show_name no)
+			(do_not_autoplace no)
+			(effects
+				(font
+					(size 1.27 1.27)
+				)
+				(justify left)
+			)
+		)
+		(property "Value" "R10k"
+			(at 46.99 44.4499 0)
+			(show_name no)
+			(do_not_autoplace no)
+			(effects
+				(font
+					(size 1.27 1.27)
+				)
+				(justify left)
+			)
+		)
+		(property "Footprint" "Resistor_SMD:R_0805_2012Metric_Pad1.20x1.40mm_HandSolder"
+			(at 42.672 43.18 90)
+			(hide yes)
+			(show_name no)
+			(do_not_autoplace no)
+			(effects
+				(font
+					(size 1.27 1.27)
+				)
+			)
+		)
+		(property "Datasheet" ""
+			(at 44.45 43.18 0)
+			(hide yes)
+			(show_name no)
+			(do_not_autoplace no)
+			(effects
+				(font
+					(size 1.27 1.27)
+				)
+			)
+		)
+		(property "Description" "Resistor"
+			(at 44.45 43.18 0)
+			(hide yes)
+			(show_name no)
+			(do_not_autoplace no)
+			(effects
+				(font
+					(size 1.27 1.27)
+				)
+			)
+		)
+		(pin "1"
+		)
+		(pin "2"
+		)
+		(instances
+			(project "PD65W_Charger"
+				(path "/f68aa78b-d8fe-48c9-a9fd-167d27b7d44f"
+					(reference "R1")
+					(unit 1)
+				)
+			)
+		)
+	)
+	(symbol
 		(lib_id "Connector:Barrel_Jack_MountingPin")
 		(at 205.74 41.91 0)
@@
 	(symbol
 		(lib_id "Device:R")
-		(at 44.45 43.18 0)
+		(at 71.12 43.18 0)
 		(unit 1)
 		(body_style 1)
@@
 		(fields_autoplaced yes)
 		(property "Reference" "R2"
-			(at 46.99 41.9099 0)
+			(at 73.66 41.9099 0)
 			(show_name no)
 			(do_not_autoplace no)
@@
 		)
 		(property "Value" "R10k"
-			(at 46.99 44.4499 0)
+			(at 73.66 44.4499 0)
 			(show_name no)
 			(do_not_autoplace no)
@@
 		)
 		(property "Footprint" "Resistor_SMD:R_0805_2012Metric_Pad1.20x1.40mm_HandSolder"
-			(at 42.672 43.18 90)
+			(at 69.342 43.18 90)
 			(hide yes)
 			(show_name no)
@@
 		)
 		(property "Datasheet" ""
-			(at 44.45 43.18 0)
+			(at 71.12 43.18 0)
 			(hide yes)
 			(show_name no)
@@
 		)
 		(property "Description" "Resistor"
-			(at 44.45 43.18 0)
+			(at 71.12 43.18 0)
 			(hide yes)
 			(show_name no)
@@
 					(unit 1)
 				)
-			)
-		)
-	)
-	(symbol
-		(lib_id "Device:R")
-		(at 71.12 43.18 0)
-		(unit 1)
-		(body_style 1)
-		(exclude_from_sim no)
-		(in_bom yes)
-		(on_board yes)
-		(in_pos_files yes)
-		(dnp no)
-		(fields_autoplaced yes)
-		(property "Reference" "R1"
-			(at 73.66 41.9099 0)
-			(show_name no)
-			(do_not_autoplace no)
-			(effects
-				(font
-					(size 1.27 1.27)
-				)
-				(justify left)
-			)
-		)
-		(property "Value" "R10k"
-			(at 73.66 44.4499 0)
-			(show_name no)
-			(do_not_autoplace no)
-			(effects
-				(font
-					(size 1.27 1.27)
-				)
-				(justify left)
-			)
-		)
-		(property "Footprint" "Resistor_SMD:R_0805_2012Metric_Pad1.20x1.40mm_HandSolder"
-			(at 69.342 43.18 90)
-			(hide yes)
-			(show_name no)
-			(do_not_autoplace no)
-			(effects
-				(font
-					(size 1.27 1.27)
-				)
-			)
-		)
-		(property "Datasheet" ""
-			(at 71.12 43.18 0)
-			(hide yes)
-			(show_name no)
-			(do_not_autoplace no)
-			(effects
-				(font
-					(size 1.27 1.27)
-				)
-			)
-		)
-		(property "Description" "Resistor"
-			(at 71.12 43.18 0)
-			(hide yes)
-			(show_name no)
-			(do_not_autoplace no)
-			(effects
-				(font
-					(size 1.27 1.27)
-				)
-			)
-		)
-		(pin "1"
-		)
-		(pin "2"
-		)
-		(instances
-			(project "PD65W_Charger"
-				(path "/f68aa78b-d8fe-48c9-a9fd-167d27b7d44f"
-					(reference "R1")
-					(unit 1)
-				)
